Commit message: Changed parameters according to actual robot

File: hase_description/urdf/hase.urdf.xacro (robot description, xacro)
@@ -15,5 +15,5 @@
       -->
     <joint name="base_joint" type="fixed">
-      <origin xyz="0 0 0.0102" rpy="0 0 0" />
+      <origin xyz="0 0 0.0435" rpy="0 0 0" />
       <parent link="base_footprint"/>
       <child link="base_link" />
@@ -22,8 +22,8 @@
       <visual>
         <geometry>
-          <cylinder length="0.1" radius="0.175"/>
+          <cylinder length="0.005" radius="0.175"/>
         </geometry>
         <xacro:insert_block name="material_light_grey"/>
-        <origin xyz="0.001 0 0.05199" rpy="0 0 0"/>
+        <origin xyz="0.00 0 0.0" rpy="0 0 0"/>
       </visual>
       <collision>
@@ -51,5 +51,5 @@
       <parent link="base_link"/>
       <child link="wheel_left_link"/>
-      <origin xyz="0.00 ${0.23/2} 0.0250" rpy="${-M_PI/2} 0 0"/>
+      <origin xyz="0.00 ${0.23/2} 0.0184" rpy="${-M_PI/2} 0 0"/>
       <axis xyz="0 0 1"/>
     </joint>
@@ -79,5 +79,5 @@
       <parent link="base_link"/>
       <child link="wheel_right_link"/>
-      <origin xyz="0.00 -${0.23/2} 0.0250" rpy="${-M_PI/2} 0 0"/>
+      <origin xyz="0.00 -${0.23/2} 0.0184" rpy="${-M_PI/2} 0 0"/>
       <axis xyz="0 0 1"/>
     </joint>

Commit message: Minor fixes based on catkin_lint and typos

File: hase_description/urdf/hase.urdf.xacro (robot description, xacro)
@@ -2,16 +2,8 @@
 <robot name="hase" xmlns:xacro="http://ros.org/wiki/xacro">
   <xacro:include filename="$(find hase_description)/urdf/common_properties.urdf.xacro"/>
+  <xacro:include filename="$(find hase_description)/urdf/hase_gazebo.urdf.xacro"/>
   <!-- Hase -->
   <xacro:macro name="hase">
     <link name="base_footprint"/>
-    <!--
-       Base link is set at the bottom of the base mould.
-       This is done to be compatible with the way base link
-       was configured for turtlebot 1. Refer to
-       https://github.com/turtlebot/turtlebot/issues/40
-       To put the base link at the more oft used wheel
-       axis, set the z-distance from the base_footprint
-       to 0.352.
-      -->
     <joint name="base_joint" type="fixed">
       <origin xyz="0 0 0.0435" rpy="0 0 0" />
@@ -22,7 +14,6 @@
       <visual>
         <geometry>
-          <cylinder length="0.005" radius="0.175"/>
+          <mesh filename="package://hase_description/meshes/base.dae" scale=".001 .001 .001"/>
         </geometry>
-        <xacro:insert_block name="material_light_grey"/>
         <origin xyz="0.00 0 0.0" rpy="0 0 0"/>
       </visual>
@@ -36,5 +27,5 @@
         <origin xyz="0.01 0 0"/>
         <mass value="2.4"/> <!-- 2.4/2.6 kg for small/big battery pack -->
-        <!-- Kobuki's inertia tensor is approximated by a cylinder with homogeneous mass distribution
+        <!-- Hase's inertia tensor is approximated by a cylinder with homogeneous mass distribution
              More details: http://en.wikipedia.org/wiki/List_of_moment_of_inertia_tensors
              m = 2.4 kg; h = 0.09 m; r = 0.175 m
@@ -57,7 +48,6 @@
       <visual>
         <geometry>
-          <cylinder length="0.0206" radius="0.0619125"/>
+          <mesh filename="package://hase_description/meshes/wheel.dae" scale=".001 .001 .001"/>
         </geometry>
-        <xacro:insert_block name="material_dark_grey"/>
         <origin xyz="0 0 0" rpy="0 0 0"/>
       </visual>
@@ -85,7 +75,6 @@
       <visual>
         <geometry>
-          <cylinder length="0.0206" radius="0.0619125"/>
+          <mesh filename="package://hase_description/meshes/wheel.dae" scale=".001 .001 .001"/>
         </geometry>
-        <xacro:insert_block name="material_dark_grey"/>
         <origin xyz="0 0 0" rpy="0 0 0"/>
       </visual>
@@ -104,4 +93,60 @@
       </inertial>
     </link>
+    <joint name="caster_front_joint" type="fixed">
+      <parent link="base_link"/>
+      <child link="caster_front_link"/>
+      <origin xyz="0.135 0.0 -0.021" rpy="${-M_PI/2} 0 0"/>
+    </joint>
+    <link name="caster_front_link">
+      <visual>
+        <geometry>
+          <cylinder length="0.0176" radius="0.0225"/>
+        </geometry>
+        <xacro:insert_block name="material_dark_grey"/>
+        <origin xyz="0 0 0" rpy="0 0 0"/>
+      </visual>
+      <collision>
+        <geometry>
+          <cylinder length="0.0176" radius="0.0225"/>
+        </geometry>
+        <origin rpy="0 0 0" xyz="0 0 0"/>
+      </collision>
+      <inertial>
+        <mass value="0.01" />
+        <origin xyz="0 0 0" />
+        <inertia ixx="0.001" ixy="0.0" ixz="0.0"
+                 iyy="0.001" iyz="0.0"
+                 izz="0.001" />
+      </inertial>
+    </link>
+    <joint name="caster_back_joint" type="fixed">
+      <parent link="base_link"/>
+      <child link="caster_back_link"/>
+      <origin xyz="-0.135 0.0 -0.021" rpy="${-M_PI/2} 0 0"/>
+    </joint>
+    <link name="caster_back_link">
+      <visual>
+        <geometry>
+          <cylinder length="0.0176" radius="0.0225"/>
+        </geometry>
+        <xacro:insert_block name="material_dark_grey"/>
+        <origin xyz="0 0 0" rpy="0 0 0"/>
+      </visual>
+      <collision>
+        <geometry>
+          <cylinder length="0.0176" radius="0.0225"/>
+        </geometry>
+        <origin rpy="0 0 0" xyz="0 0 0"/>
+      </collision>
+      <inertial>
+        <mass value="0.01" />
+        <origin xyz="0 0 0" />
+        <inertia ixx="0.001" ixy="0.0" ixz="0.0"
+                 iyy="0.001" iyz="0.0"
+                 izz="0.001" />
+      </inertial>
+    </link>
+    <!-- Hase Gazebo simulation details -->
+    <hase_sim/>
   </xacro:macro>
 </robot>

Commit message: Fixed base orientation (Maybe need to fix this in the freecad design)

File: hase_description/urdf/hase.urdf.xacro (robot description, xacro)
@@ -16,5 +16,5 @@
           <mesh filename="package://hase_description/meshes/base.dae" scale=".001 .001 .001"/>
         </geometry>
-        <origin xyz="0.00 0 0.0" rpy="0 0 0"/>
+        <origin xyz="0.00 0 0.0" rpy="0 0 ${M_PI/2}"/>
       </visual>
       <collision>

Commit message: Changed robot meshes and reflect in urdf

File: hase_description/urdf/hase.urdf.xacro (robot description, xacro)
@@ -7,5 +7,5 @@
     <link name="base_footprint"/>
     <joint name="base_joint" type="fixed">
-      <origin xyz="0 0 0.0435" rpy="0 0 0" />
+      <origin xyz="0 0 0.0425" rpy="0 0 0" />
       <parent link="base_footprint"/>
       <child link="base_link" />
@@ -16,10 +16,11 @@
           <mesh filename="package://hase_description/meshes/base.dae" scale=".001 .001 .001"/>
         </geometry>
-        <origin xyz="0.00 0 0.0" rpy="0 0 ${M_PI/2}"/>
+        <origin xyz="0.001 0 0.1620" rpy="0 0 0"/>
       </visual>
       <collision>
         <geometry>
-          <cylinder length="0.10938" radius="0.178"/>
+          <cylinder length="0.1" radius="0.178"/>
         </geometry>
+        <origin xyz="0.0 0 0.0435" rpy="0 0 0"/>
       </collision>
       <inertial>
@@ -42,5 +43,5 @@
       <parent link="base_link"/>
       <child link="wheel_left_link"/>
-      <origin xyz="0.00 ${0.23/2} 0.0184" rpy="${-M_PI/2} 0 0"/>
+      <origin xyz="0.00 ${0.23/2} 0.019" rpy="${-M_PI/2} 0 0"/>
       <axis xyz="0 0 1"/>
     </joint>
@@ -54,5 +55,5 @@
       <collision>
         <geometry>
-          <cylinder length="0.0206" radius="0.0619125"/>
+          <cylinder length="0.0205" radius="0.0617"/>
         </geometry>
         <origin rpy="0 0 0" xyz="0 0 0"/>
@@ -69,5 +70,5 @@
       <parent link="base_link"/>
       <child link="wheel_right_link"/>
-      <origin xyz="0.00 -${0.23/2} 0.0184" rpy="${-M_PI/2} 0 0"/>
+      <origin xyz="0.00 -${0.23/2} 0.019" rpy="${-M_PI/2} 0 0"/>
       <axis xyz="0 0 1"/>
     </joint>
@@ -81,5 +82,5 @@
       <collision>
         <geometry>
-          <cylinder length="0.0206" radius="0.0619125"/>
+          <cylinder length="0.0205" radius="0.0615"/>
         </geometry>
         <origin rpy="0 0 0" xyz="0 0 0"/>
@@ -96,17 +97,10 @@
       <parent link="base_link"/>
       <child link="caster_front_link"/>
-      <origin xyz="0.135 0.0 -0.021" rpy="${-M_PI/2} 0 0"/>
+      <origin xyz="0.115 0.0 0.0065" rpy="${-M_PI/2} 0 0"/>
     </joint>
     <link name="caster_front_link">
-      <visual>
-        <geometry>
-          <cylinder length="0.0176" radius="0.0225"/>
-        </geometry>
-        <xacro:insert_block name="material_dark_grey"/>
-        <origin xyz="0 0 0" rpy="0 0 0"/>
-      </visual>
       <collision>
         <geometry>
-          <cylinder length="0.0176" radius="0.0225"/>
+          <cylinder length="0.0176" radius="0.05"/>
         </geometry>
         <origin rpy="0 0 0" xyz="0 0 0"/>
@@ -123,17 +117,10 @@
       <parent link="base_link"/>
       <child link="caster_back_link"/>
-      <origin xyz="-0.135 0.0 -0.021" rpy="${-M_PI/2} 0 0"/>
+      <origin xyz="-0.135 0.0 0.0095" rpy="${-M_PI/2} 0 0"/>
     </joint>
     <link name="caster_back_link">
-      <visual>
-        <geometry>
-          <cylinder length="0.0176" radius="0.0225"/>
-        </geometry>
-        <xacro:insert_block name="material_dark_grey"/>
-        <origin xyz="0 0 0" rpy="0 0 0"/>
-      </visual>
       <collision>
         <geometry>
-          <cylinder length="0.0176" radius="0.0225"/>
+          <cylinder length="0.0176" radius="0.05"/>
         </geometry>
         <origin rpy="0 0 0" xyz="0 0 0"/>

Commit message: Fixed physical issues in the simulator

File: hase_description/urdf/hase.urdf.xacro (robot description, xacro)
@@ -7,5 +7,5 @@
     <link name="base_footprint"/>
     <joint name="base_joint" type="fixed">
-      <origin xyz="0 0 0.0425" rpy="0 0 0" />
+      <origin xyz="0 0 0.0402" rpy="0 0 0" />
       <parent link="base_footprint"/>
       <child link="base_link" />
@@ -16,5 +16,5 @@
           <mesh filename="package://hase_description/meshes/base.dae" scale=".001 .001 .001"/>
         </geometry>
-        <origin xyz="0.001 0 0.1620" rpy="0 0 0"/>
+        <origin xyz="0 0 0.0548" rpy="0 0 0"/>
       </visual>
       <collision>
@@ -22,9 +22,9 @@
           <cylinder length="0.1" radius="0.178"/>
         </geometry>
-        <origin xyz="0.0 0 0.0435" rpy="0 0 0"/>
+        <origin xyz="0.0 0 0.0548" rpy="0 0 0"/>
       </collision>
       <inertial>
         <!-- COM experimentally determined -->
-        <origin xyz="0.01 0 0"/>
+        <origin xyz="0 0 0"/>
         <mass value="2.4"/> <!-- 2.4/2.6 kg for small/big battery pack -->
         <!-- Hase's inertia tensor is approximated by a cylinder with homogeneous mass distribution
@@ -43,5 +43,5 @@
       <parent link="base_link"/>
       <child link="wheel_left_link"/>
-      <origin xyz="0.00 ${0.23/2} 0.019" rpy="${-M_PI/2} 0 0"/>
+      <origin xyz="0.00 ${0.23/2} 0.0213" rpy="${-M_PI/2} 0 0"/>
       <axis xyz="0 0 1"/>
     </joint>
@@ -55,10 +55,10 @@
       <collision>
         <geometry>
-          <cylinder length="0.0205" radius="0.0617"/>
+          <cylinder length="0.0205" radius="0.0615"/>
         </geometry>
         <origin rpy="0 0 0" xyz="0 0 0"/>
       </collision>
       <inertial>
-        <mass value="0.01" />
+        <mass value="0.1" />
         <origin xyz="0 0 0" />
         <inertia ixx="0.001" ixy="0.0" ixz="0.0"
@@ -70,5 +70,5 @@
       <parent link="base_link"/>
       <child link="wheel_right_link"/>
-      <origin xyz="0.00 -${0.23/2} 0.019" rpy="${-M_PI/2} 0 0"/>
+      <origin xyz="0.00 -${0.23/2} 0.0213" rpy="${-M_PI/2} 0 0"/>
       <axis xyz="0 0 1"/>
     </joint>
@@ -87,5 +87,5 @@
       </collision>
       <inertial>
-        <mass value="0.01" />
+        <mass value="0.1" />
         <origin xyz="0 0 0" />
         <inertia ixx="0.001" ixy="0.0" ixz="0.0"
@@ -97,10 +97,10 @@
       <parent link="base_link"/>
       <child link="caster_front_link"/>
-      <origin xyz="0.115 0.0 0.0065" rpy="${-M_PI/2} 0 0"/>
+      <origin xyz="0.115 0.0 0.015" rpy="${-M_PI/2} 0 0"/>
     </joint>
     <link name="caster_front_link">
       <collision>
         <geometry>
-          <cylinder length="0.0176" radius="0.05"/>
+          <cylinder length="0.015" radius="0.055"/>
         </geometry>
         <origin rpy="0 0 0" xyz="0 0 0"/>
@@ -117,10 +117,10 @@
       <parent link="base_link"/>
       <child link="caster_back_link"/>
-      <origin xyz="-0.135 0.0 0.0095" rpy="${-M_PI/2} 0 0"/>
+      <origin xyz="-0.115 0.0 0.015" rpy="${-M_PI/2} 0 0"/>
     </joint>
     <link name="caster_back_link">
       <collision>
         <geometry>
-          <cylinder length="0.0176" radius="0.05"/>
+          <cylinder length="0.015" radius="0.055"/>
         </geometry>
         <origin rpy="0 0 0" xyz="0 0 0"/>

Commit message: Changed urdf parameters to reflect the real robot

File: hase_description/urdf/hase.urdf.xacro (robot description, xacro)
@@ -7,5 +7,5 @@
     <link name="base_footprint"/>
     <joint name="base_joint" type="fixed">
-      <origin xyz="0 0 0.0402" rpy="0 0 0" />
+      <origin xyz="0 0 0.0252" rpy="0 0 0" />
       <parent link="base_footprint"/>
       <child link="base_link" />
@@ -43,5 +43,5 @@
       <parent link="base_link"/>
       <child link="wheel_left_link"/>
-      <origin xyz="0.00 ${0.23/2} 0.0213" rpy="${-M_PI/2} 0 0"/>
+      <origin xyz="0.00 ${0.23/2} 0.0363" rpy="${-M_PI/2} 0 0"/>
       <axis xyz="0 0 1"/>
     </joint>
@@ -70,5 +70,5 @@
       <parent link="base_link"/>
       <child link="wheel_right_link"/>
-      <origin xyz="0.00 -${0.23/2} 0.0213" rpy="${-M_PI/2} 0 0"/>
+      <origin xyz="0.00 -${0.23/2} 0.0363" rpy="${-M_PI/2} 0 0"/>
       <axis xyz="0 0 1"/>
     </joint>
@@ -102,5 +102,5 @@
       <collision>
         <geometry>
-          <cylinder length="0.015" radius="0.055"/>
+          <cylinder length="0.015" radius="0.04"/>
         </geometry>
         <origin rpy="0 0 0" xyz="0 0 0"/>
@@ -122,5 +122,5 @@
       <collision>
         <geometry>
-          <cylinder length="0.015" radius="0.055"/>
+          <cylinder length="0.015" radius="0.04"/>
         </geometry>
         <origin rpy="0 0 0" xyz="0 0 0"/>
