Commit message: First test to add kinect sensor

File: hase_description/urdf/hase_gazebo.urdf.xacro (robot description, xacro)
@@ -39,3 +39,41 @@
     </gazebo>
   </xacro:macro>
+  <xacro:macro name="turtlebot_sim_3dsensor">
+    <gazebo reference="camera_link">
+      <sensor type="depth" name="camera">
+        <always_on>true</always_on>
+        <update_rate>20.0</update_rate>
+        <camera>
+          <horizontal_fov>${60.0*M_PI/180.0}</horizontal_fov>
+          <image>
+            <format>R8G8B8</format>
+            <width>640</width>
+            <height>480</height>
+          </image>
+          <clip>
+            <near>0.05</near>
+            <far>8.0</far>
+          </clip>
+        </camera>
+        <plugin name="kinect_camera_controller" filename="libgazebo_ros_openni_kinect.so">
+          <cameraName>camera</cameraName>
+          <alwaysOn>true</alwaysOn>
+          <updateRate>10</updateRate>
+          <imageTopicName>rgb/image_raw</imageTopicName>
+          <depthImageTopicName>depth/image_raw</depthImageTopicName>
+          <pointCloudTopicName>depth/points</pointCloudTopicName>
+          <cameraInfoTopicName>rgb/camera_info</cameraInfoTopicName>
+          <depthImageCameraInfoTopicName>depth/camera_info</depthImageCameraInfoTopicName>
+          <frameName>camera_depth_optical_frame</frameName>
+          <baseline>0.1</baseline>
+          <distortion_k1>0.0</distortion_k1>
+          <distortion_k2>0.0</distortion_k2>
+          <distortion_k3>0.0</distortion_k3>
+          <distortion_t1>0.0</distortion_t1>
+          <distortion_t2>0.0</distortion_t2>
+          <pointCloudCutoff>0.4</pointCloudCutoff>
+        </plugin>
+      </sensor>
+    </gazebo>
+  </xacro:macro>
 </robot>

Commit message: Fixed some issues with package names

File: hase_description/urdf/hase_gazebo.urdf.xacro (robot description, xacro)
@@ -39,5 +39,5 @@
     </gazebo>
   </xacro:macro>
-  <xacro:macro name="turtlebot_sim_3dsensor">
+  <xacro:macro name="hase_sim_3dsensor">
     <gazebo reference="camera_link">
       <sensor type="depth" name="camera">

File: hase_description/urdf/sensors/kinect.urdf.xacro (robot description, xacro)
@@ -1,7 +1,7 @@
 <?xml version="1.0"?>
 <robot name="sensor_kinect" xmlns:xacro="http://ros.org/wiki/xacro">
-  <xacro:include filename="$(find turtlebot_description)/urdf/turtlebot_gazebo.urdf.xacro"/>
-  <xacro:include filename="$(find turtlebot_description)/urdf/turtlebot_properties.urdf.xacro"/>
-  <!-- Parameterised in part by the values in turtlebot_properties.urdf.xacro -->
+  <xacro:include filename="$(find hase_description)/urdf/hase_gazebo.urdf.xacro"/>
+<!--  <xacro:include filename="$(find hase_description)/urdf/hase_properties.urdf.xacro"/>-->
+  <!-- Parameterised in part by the values in hase_properties.urdf.xacro -->
   <xacro:macro name="sensor_kinect" params="parent">
     <joint name="camera_rgb_joint" type="fixed">
@@ -42,5 +42,5 @@
      <origin xyz="0 0 0" rpy="0 0 ${M_PI/2}"/>
       <geometry>
-       <mesh filename="package://turtlebot_description/meshes/sensors/kinect.dae"/>
+       <mesh filename="package://hase_description/meshes/sensors/kinect.dae"/>
       </geometry>
     </visual>
@@ -91,5 +91,5 @@
 	</link>
 	<!-- Kinect sensor for simulation -->
-	<turtlebot_sim_3dsensor/>
+	<hase_sim_3dsensor/>
   </xacro:macro>
 </robot>
